File: CheeseShield/CheeseShield.sch (KiCad schematic (older format))
At the start: 32 parts, among them J1 MS3 Toggle, J10 BlueTooth Connection, J2 MS2 Toggle, J3 MS1 Toggle, J4 Power Screw Terminal, J5 JST XH_Stepper, J6 Temp1 3PinFan, J7 TempBed 3PinFan, J8 Temp0 3PinFan, J9 SSR Connection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

Commit message: feat: updated circuit to minimize servo jitter
Parts:
- removed J10: BlueTooth Connection, symbol Connector:Conn_01x04_Female
- removed J5: JST XH_Stepper, Connectors_JST:JST_XH_B04B-XH-A_04x2.50mm_Straight, symbol Connector:Conn_01x04_Female
- removed J?: Servo_0 Header, symbol Connector:Conn_01x03_Female
- removed J?: Servo_1 Header, symbol Connector:Conn_01x03_Female
- removed J?: Servo_2 Header, symbol Connector:Conn_01x03_Female
- removed J?: Servo_3 Header, symbol Connector:Conn_01x03_Female
- added J10: Conn_01x05, Connector_PinHeader_2.54mm:PinHeader_1x05_P2.54mm_Vertical, symbol Connector_Generic:Conn_01x05
- added J5: Conn_02x10_Odd_Even, Connector_IDC:IDC-Header_2x10_P2.54mm_Vertical, symbol Connector_Generic:Conn_02x10_Odd_Even
- added U1: LevelConverter, TomsPartsLibrary:LevelConverter, symbol TomsPartsLibrary:LevelConverter
Connections:
- net labels added: 1A, 1B, 2A, 2B
- wire segments 178 -> 167
- no-connect marks 7 -> 11
Other:
- moved on the sheet: J6, J7, J8, J9, M1, R1, R2, R3
